Commit message: Freeze current arm control implementation

File: gui/public/assets/kinematics/arm.urdf (robot description, URDF)
Before this commit: robot robot_arm, 8 links, 7 joints
Links:
- added link j4_pivot_link
Joints:
- added joint j4_pivot_joint: type fixed, parent arm2, child j4_pivot_link, origin xyz=0 0.05 0.6 rpy=0 0 0

File: test/moveit2/arm_moveit_config/config/arm.urdf (robot description, URDF)
Before this commit: robot robot_arm, 8 links, 7 joints
Links:
- added link j4_pivot_link
Joints:
- added joint j4_pivot_joint: type fixed, parent arm2, child j4_pivot_link, origin xyz=0 0.05 0.6 rpy=0 0 0
