Commit message: Make position arm control MoveIt2-only

File: test/moveit2/arm_moveit_config/config/arm.urdf (robot description, URDF)
Before this commit: robot robot_arm, 9 links, 8 joints
Joints:
- joint yaw_joint: origin xyz=0 0.05 0.6 rpy=0 0 0 -> xyz=0 0 0 rpy=0 0 0; parent arm2 -> j4_pivot_link
