Commit message: Restored pitch joint limits and separeate encoder turn-reference flag

File: basestation/arm_moveit_config/config/arm.urdf (robot description, URDF)
Before this commit: robot robot_arm, 9 links, 8 joints
Joints:
- joint pitch_joint: limit lower=-0.0873 upper=4.7997 effort=100 velocity=1.0 -> lower=-0.0873 upper=3.7525 effort=100 velocity=1.0

File: gui/public/assets/kinematics/arm.urdf (robot description, URDF)
Before this commit: robot robot_arm, 9 links, 8 joints
Joints:
- joint pitch_joint: limit lower=-0.0873 upper=4.7997 effort=100 velocity=1.0 -> lower=-0.0873 upper=3.7525 effort=100 velocity=1.0

File: rover/control/arm/rover_ws/src/dcr_arm_driver/urdf/robot_arm.urdf (robot description, URDF)
Before this commit: robot robot_arm, 9 links, 8 joints
Joints:
- joint pitch_joint: limit lower=-0.0873 upper=4.7997 effort=100 velocity=1.0 -> lower=-0.0873 upper=3.7525 effort=100 velocity=1.0
